File: PCB/stock/stock_v2/stock_v2.kicad_sch (KiCad schematic)
At the start: 24 parts, among them J1 Conn_01x02, J2 Conn_01x02, J3 Conn_01x02, J4 Conn_01x03, J5 Conn_01x02, J6 Conn_01x02, J7 Conn_01x02, U1 LM358, U2 LM741, U3 LM358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

Commit message: tudo ok
se e fd pcb ok
Connections:
- net +9V: no longer C2.1, J4.3 (Pin_3), U1.8 (V+), U3.8 (V+), U6.1 (IN)
- net -9V: no longer J4.1 (Pin_1), U1.4 (V-), U3.4 (V-)
- new net +12V: J4.1 (Pin_1), U1.8 (V+), U3.8 (V+)
- new net -12V: C2.1, J4.3 (Pin_3), U1.4 (V-), U3.4 (V-), U6.1 (IN)
Other:
- note added: "1"
- note added: "2"
- note added: "3"
- note added: "4"
- note added: "5"
- company: (none) -> UFPel
- title: (none) -> Potenciostato Single-Ended
- moved on the sheet: C1, C2, C4, J4, U1C, U3C, U6
